File: hardware/eMMC dumper.kicad_sch (KiCad schematic)
At the start: 25 parts, among them J1 Micro_SD_Card, J2 USB_B_Micro, U4 EMMC04G-M627-A01

Commit message: Moved LEDs, renamed testpoints
Parts:
- renumbered TP5 to 1V2, TP4 to 3V3, TP2 to CLK, TP1 to CMD, TP3 to D0, TP8 to GND1, TP7 to U_RX1, TP6 to U_TX1
Changed lines of the file:
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@@
 		(on_board yes)
 		(dnp no)
-		(fields_autoplaced yes)
 		(property "Reference" "D1"
-			(at 221.2975 91.44 0)
+			(at 215.138 94.234 0)
 			(effects
 				(font
@@
 		)
 		(property "Value" "LED"
-			(at 221.2975 93.98 0)
+			(at 215.138 96.774 0)
 			(effects
 				(font
@@
 		(dnp no)
 		(fields_autoplaced yes)
-		(property "Reference" "TP2"
+		(property "Reference" "CLK"
 			(at 153.67 126.9999 90)
 			(effects
@@
 			(project "eMMC dumper"
 				(path "/70144d06-8877-4e78-ba5e-b83edad21557"
-					(reference "TP2")
+					(reference "CLK")
 					(unit 1)
 				)
@@
 		(on_board yes)
 		(dnp no)
-		(fields_autoplaced yes)
-		(property "Reference" "TP1"
-			(at 158.75 124.4599 90)
+		(property "Reference" "CMD"
+			(at 158.496 124.46 90)
 			(effects
 				(font
@@
 			(project ""
 				(path "/70144d06-8877-4e78-ba5e-b83edad21557"
-					(reference "TP1")
+					(reference "CMD")
 					(unit 1)
 				)
@@
 		(dnp no)
 		(property "Reference" "D2"
-			(at 220.98 106.934 0)
+			(at 215.138 100.584 0)
 			(effects
 				(font
@@
 		)
 		(property "Value" "LED"
-			(at 220.98 109.22 0)
+			(at 215.138 102.87 0)
 			(effects
 				(font
@@
 		(on_board yes)
 		(dnp no)
-		(fields_autoplaced yes)
 		(property "Reference" "D3"
-			(at 221.2975 101.6 0)
+			(at 215.138 105.41 0)
 			(effects
 				(font
@@
 		)
 		(property "Value" "LED"
-			(at 221.2975 104.14 0)
+			(at 215.138 107.95 0)
 			(effects
 				(font
@@
 		(dnp no)
 		(property "Reference" "D4"
-			(at 220.98 117.094 0)
+			(at 215.138 110.998 0)
 			(effects
 				(font
@@
 		)
 		(property "Value" "LED"
-			(at 220.98 119.38 0)
+			(at 215.138 113.284 0)
 			(effects
 				(font
@@
 		(on_board yes)
 		(dnp no)
-		(property "Reference" "TP5"
+		(property "Reference" "1V2"
 			(at 139.954 60.452 0)
 			(effects
@@
 			(project "eMMC dumper"
 				(path "/70144d06-8877-4e78-ba5e-b83edad21557"
-					(reference "TP5")
+					(reference "1V2")
 					(unit 1)
 				)
@@
 		(dnp no)
 		(fields_autoplaced yes)
-		(property "Reference" "TP3"
+		(property "Reference" "D0"
 			(at 148.59 129.5399 90)
 			(effects
@@
 			(project "eMMC dumper"
 				(path "/70144d06-8877-4e78-ba5e-b83edad21557"
-					(reference "TP3")
+					(reference "D0")
 					(unit 1)
 				)
@@
 		(on_board yes)
 		(dnp no)
-		(property "Reference" "TP8"
+		(property "Reference" "GND1"
 			(at 200.66 72.39 90)
 			(effects
@@
 			(project "eMMC dumper"
 				(path "/70144d06-8877-4e78-ba5e-b83edad21557"
-					(reference "TP8")
+					(reference "GND1")
 					(unit 1)
 				)
@@
 		(on_board yes)
 		(dnp no)
-		(property "Reference" "TP6"
+		(property "Reference" "U_TX1"
 			(at 200.66 67.31 90)
 			(effects
@@
 			(project "eMMC dumper"
 				(path "/70144d06-8877-4e78-ba5e-b83edad21557"
-					(reference "TP6")
+					(reference "U_TX1")
 					(unit 1)
 				)
@@
 		(on_board yes)
 		(dnp no)
-		(property "Reference" "TP4"
+		(property "Reference" "3V3"
 			(at 200.66 64.77 90)
 			(effects
@@
 			(project "eMMC dumper"
 				(path "/70144d06-8877-4e78-ba5e-b83edad21557"
-					(reference "TP4")
+					(reference "3V3")
 					(unit 1)
 				)
@@
 		(on_board yes)
 		(dnp no)
-		(fields_autoplaced yes)
 		(property "Reference" "#PWR016"
 			(at 146.05 59.69 0)
@@
 		)
 		(property "Value" "+3V3"
-			(at 146.05 50.8 0)
+			(at 143.002 51.054 0)
 			(effects
 				(font
 					(size 1.27 1.27)
 				)
+				(justify left)
 			)
 		)
@@
 		(on_board yes)
 		(dnp no)
-		(property "Reference" "TP7"
+		(property "Reference" "U_RX1"
 			(at 200.66 69.85 90)
 			(effects
@@
 			(project "eMMC dumper"
 				(path "/70144d06-8877-4e78-ba5e-b83edad21557"
-					(reference "TP7")
+					(reference "U_RX1")
 					(unit 1)
 				)
